File: beer.brd (EAGLE design)
At the start: 55.9 x 55.9 mm, 47 parts, among them IC3 TPS77350, K1 RT184005, Q1 2N2222, U5 ATMEGA32U4-XUAU, X2 USB-MICROB, Y1 16MHz KX-7

Commit message: Initial routing complete
Parts:
- removed L2: MH2029-300Y, wuerth-elektronik:0805
- removed Q1: 2N2222, transistor-small-signal:TO18A
- added JP1: (no value), SparkFun:1X04
- added Q2: TIP120, transistor-power:TO220AH
- moved FAN_OUT 139.6 mm to (29.9, 61.0), turned to 180 degrees
- moved R2 117.3 mm to (12.9, 47.1), turned to 270 degrees
- moved PELTIER 113.2 mm to (27.3, 70.0)
- moved K1 109.9 mm to (42.3, 58.3), turned to 90 degrees
- moved D1 106.1 mm to (25.8, 46.5)
- moved C1 94.4 mm to (27.4, 65.3), turned to 90 degrees
- moved C6 93.2 mm to (29.1, 65.3), turned to 270 degrees
- moved R1 58.0 mm to (38.0, 31.6), turned to 180 degrees
- moved JP3 54.3 mm to (8.23, 45.0), turned to 90 degrees
- moved C24 42.5 mm to (22.9, 2.54), turned to 270 degrees
- moved IC3 38.1 mm to (14.7, 5.03), turned to 270 degrees
- moved D2 38.1 mm to (18.9, 40.4)
- moved C28 35.6 mm to (7.21, 41.2)
- moved C27 35.5 mm to (27.1, 42.1), turned to 0 degrees
- moved C26 34.1 mm to (34.3, 31.6), turned to 180 degrees
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Connections:
- removed net D4: U5.25
- removed net D7: U5.1
- removed net IO11*: U5.12
- removed net MOT/SENS_1: U5.36
- removed net MOT/SENS_2: U5.37
- removed net MOT/SENS_3: U5.38
- removed net MOT/SENS_4: U5.39
- removed net MOT/SENS_5: U5.40
- removed net MOT/SENS_6: U5.41
- removed net REC3: U5.28
- removed net REC4: U5.29
- removed net REC5: U5.30
- removed net REC6: U5.31
- removed net SCL5V: U5.18
- removed net SDA5V: U5.19
- new net AUX0: JP1.4, U5.12
- new net AUX1: JP1.3, U5.30
- new net AUX2: JP1.2, U5.29
- new net AUX3: JP1.1, U5.28
- net +5V: now also K1.A1; no longer K1.14
- net GND: now also Q2.E; no longer L2.2, Q1.E
- net N$1: now also K1.11; no longer K1.A2
- net N$3: now also K1.A2, Q2.C; no longer K1.11, Q1.C
- net N$7: now also Q2.B; no longer Q1.B
- net UGND: no longer L2.1
- net VCC: now also K1.14; no longer K1.A1
Routing:
- net VCC: track 0.00 -> 143.3 mm, vias 0 -> 2
- net N$5: track 0.00 -> 114.9 mm, vias 0 -> 2
- net PD2: track 11.9 -> 89.1 mm, vias 0 -> 6
- net PD1: track 12.0 -> 88.1 mm, vias 0 -> 6
- net 3V3: track 85.0 -> 11.5 mm, vias 6 -> 0
- net D-: track 6.75 -> 53.2 mm, vias 0 -> 2
- net HWB: track 2.21 -> 42.3 mm, vias 0 -> 4
- net AVCC: track 21.8 -> 59.5 mm, vias 0 -> 2
- net REC1: track 34.0 -> 0.00 mm
- net AUX0: track 0.00 -> 31.4 mm, vias 0 -> 2
- net GND: track 89.5 -> 118.5 mm, vias 24 -> 12
- net REC2: track 28.2 -> 0.00 mm
- net REC3: track 27.3 -> 0.00 mm
- net N$3: track 0.00 -> 27.1 mm
- net REC4: track 26.4 -> 0.00 mm
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- removed copper zone on layer 1, net +5V
- removed copper zone on layer 1, net 3V3
- removed copper zone on layer 1, net GND
Other:
- board size 55.9 x 55.9 mm -> 51.7 x 74.7 mm
- board text removed: "10nF"
- board text removed: "1M"
- board text removed: "220nF"
- board text removed: "AUX"
- board text removed: "CA"
- board text removed: "CB"
- board text removed: "CC"
- board text removed: "CD"
- board text removed: "CE"
- board text removed: "CF"
- board text removed: "D13"
- board text removed: "DA"
- board text removed: "FUSE"
- board text removed: "ICSP"
- board text removed: "Jan 2013"
- board text removed: "LA"
- board text removed: "PWR"
- board text removed: "Peregrine Board V1.1"
- board text removed: "RA"
- board text removed: "RA-10K RB-1K RC-22"
- board text removed: "RB"
- board text removed: "RC"
- board text removed: "RX"
- board text removed: "TX"
- board text removed: "X"
- board text removed: "Y"
- board text removed: "ZA"
