File: beer.sch (EAGLE design)
At the start: 47 parts, among them IC3 TPS77350, K1 RT184005, Q1 2N2222, U5 ATMEGA32U4-XUAU, X2 USB-MICROB, Y1 16MHz KX-7

Commit message: Initial routing complete
Parts:
- removed L2: MH2029-300Y, wuerth-elektronik:WE-CBF_0805
- removed Q1: 2N2222, transistor-small-signal:2N2222
- added JP1: (no value), SparkFun:M04PTH
- added Q2: TIP120, transistor-power:TIP120
Connections:
- removed net D4: U5.(ICP1/ADC8)PD4
- removed net D7: U5.(INT6/AIN0)PE6
- removed net IO11*: U5.(PCINT7/OC0A/OC1C/#RTS)PB7
- removed net MOT/SENS_1: U5.(ADC7/TDI)PF7
- removed net MOT/SENS_2: U5.(ADC6/TDO)PF6
- removed net MOT/SENS_3: U5.(ADC5/TMS)PF5
- removed net MOT/SENS_4: U5.(ADC4/TCK)PF4
- removed net MOT/SENS_5: U5.(ADC1)PF1
- removed net MOT/SENS_6: U5.(ADC0)PF0
- removed net REC3: U5.(ADC11/PCINT4)PB4
- removed net REC4: U5.(PCINT5/OC1A/#OC4B/ADC12)PB5
- removed net REC5: U5.(PCINT6/OC1B/OC4B/ADC13)PB6
- removed net REC6: U5.(OC3A/#0C4A)PC6
- removed net SCL5V: U5.(OC0B/SCL/INT0)PD0
- removed net SDA5V: U5.(SDA/INT1)PD1
- new net AUX0: JP1.4, U5.(PCINT7/OC0A/OC1C/#RTS)PB7
- new net AUX1: JP1.3, U5.(PCINT6/OC1B/OC4B/ADC13)PB6
- new net AUX2: JP1.2, U5.(PCINT5/OC1A/#OC4B/ADC12)PB5
- new net AUX3: JP1.1, U5.(ADC11/PCINT4)PB4
- net +5V: now also K11.1; no longer K12.S
- net GND: now also Q2.E; no longer L2.2, Q1.E
- net N$1: now also K12.P; no longer K11.2
- net N$3: now also K11.2, Q2.C; no longer K12.P, Q1.C
- net N$7: now also Q2.B; no longer Q1.B
- net UGND: no longer L2.1
- net VCC: now also K12.S; no longer K11.1
Other:
- note added: "+12V DC in"
- note added: "Aux I/O"
- note added: "TIP102"
- moved on the sheet: K1, POWER_IN
